Commit message: upload working files: migrate the xacro files and add display.launch.py

File: op3_description/urdf/robotis_op3.structure.head.xacro (robot description, xacro)
@@ -1,7 +1,4 @@
 <?xml version="1.0" ?>
 <robot xmlns:xacro="http://ros.org/wiki/xacro">
-  <!--
-  <xacro:property name="pi" value="3.141592654" />
-  -->
   <!-- head -->
   <xacro:macro name="robotis_op3_head" params="parent">
@@ -21,7 +18,7 @@
       <xacro:insert_mesh_head_pan_link />
     </visual>
-    <collision>
+    <!-- <collision>
       <xacro:insert_mesh_head_pan_link />
-    </collision>
+    </collision> -->
     <inertial>
       <xacro:insert_inertia_head_pan_link />
@@ -43,7 +40,7 @@
       <xacro:insert_mesh_head_tilt_link />
     </visual>
-    <collision>
+    <!-- <collision>
       <xacro:insert_mesh_head_tilt_link />
-    </collision>
+    </collision> -->
     <inertial>
       <xacro:insert_inertia_head_tilt_link />

File: op3_description/urdf/robotis_op3.structure.larm.xacro (robot description, xacro)
@@ -1,7 +1,4 @@
 <?xml version="1.0" ?>
 <robot xmlns:xacro="http://ros.org/wiki/xacro">
-  <!--
-  <xacro:property name="pi" value="3.141592654" />
-  -->
   <!-- left leg -->
   <xacro:macro name="robotis_op3_l_arm" params="parent">
@@ -21,7 +18,7 @@
       <xacro:insert_mesh_l_sho_pitch_link />
     </visual>
-    <collision>
+    <!-- <collision>
       <xacro:insert_mesh_l_sho_pitch_link />
-    </collision>
+    </collision> -->
     <inertial>
       <xacro:insert_inertia_l_sho_pitch_link />
@@ -43,7 +40,7 @@
       <xacro:insert_mesh_l_sho_roll_link />
     </visual>
-    <collision>
+    <!-- <collision>
       <xacro:insert_mesh_l_sho_roll_link />
-    </collision>
+    </collision> -->
     <inertial>
       <xacro:insert_inertia_l_sho_roll_link />
@@ -65,7 +62,7 @@
       <xacro:insert_mesh_l_el_link />
     </visual>
-    <collision>
+    <!-- <collision>
       <xacro:insert_mesh_l_el_link />
-    </collision>
+    </collision> -->
     <inertial>
       <xacro:insert_inertia_l_el_link />

File: op3_description/urdf/robotis_op3.structure.lleg.xacro (robot description, xacro)
@@ -1,7 +1,4 @@
 <?xml version="1.0" ?>
 <robot xmlns:xacro="http://ros.org/wiki/xacro">
-  <!--
-  <xacro:property name="pi" value="3.141592654" />
-  -->
   <!-- left leg -->
   <xacro:macro name="robotis_op3_l_leg" params="parent">
@@ -21,7 +18,7 @@
       <xacro:insert_mesh_l_hip_yaw_link />
     </visual>
-    <collision>
+    <!-- <collision>
       <xacro:insert_mesh_l_hip_yaw_link />
-    </collision>
+    </collision> -->
     <inertial>
       <xacro:insert_inertia_l_hip_yaw_link />
@@ -43,7 +40,7 @@
       <xacro:insert_mesh_l_hip_roll_link />
     </visual>
-    <collision>
+    <!-- <collision>
       <xacro:insert_mesh_l_hip_roll_link />
-    </collision>
+    </collision> -->
     <inertial>
       <xacro:insert_inertia_l_hip_roll_link />
@@ -65,7 +62,7 @@
       <xacro:insert_mesh_l_hip_pitch_link />
     </visual>
-    <collision>
+    <!-- <collision>
       <xacro:insert_mesh_l_hip_pitch_link />
-    </collision>
+    </collision> -->
     <inertial>
       <xacro:insert_inertia_l_hip_pitch_link />
@@ -87,7 +84,7 @@
       <xacro:insert_mesh_l_knee_link />
     </visual>
-    <collision>
+    <!-- <collision>
       <xacro:insert_mesh_l_knee_link />
-    </collision>
+    </collision> -->
     <inertial>
       <xacro:insert_inertia_l_knee_link />
@@ -109,7 +106,7 @@
       <xacro:insert_mesh_l_ank_pitch_link />
     </visual>
-    <collision>
+    <!-- <collision>
       <xacro:insert_mesh_l_ank_pitch_link />
-    </collision>
+    </collision> -->
     <inertial>
       <xacro:insert_inertia_l_ank_pitch_link />
@@ -131,7 +128,7 @@
       <xacro:insert_mesh_l_ank_roll_link />
     </visual>
-    <collision>
+    <!-- <collision>
       <xacro:insert_mesh_l_ank_roll_link />
-    </collision>
+    </collision> -->
     <inertial>
       <xacro:insert_inertia_l_ank_roll_link />

File: op3_description/urdf/robotis_op3.structure.rarm.xacro (robot description, xacro)
@@ -1,7 +1,4 @@
 <?xml version="1.0" ?>
 <robot xmlns:xacro="http://ros.org/wiki/xacro">
-  <!--
-  <xacro:property name="pi" value="3.141592654" />
-  -->
   <!-- right arm -->
   <xacro:macro name="robotis_op3_r_arm" params="parent">
@@ -21,7 +18,7 @@
       <xacro:insert_mesh_r_sho_pitch_link />
     </visual>
-    <collision>
+    <!-- <collision>
       <xacro:insert_mesh_r_sho_pitch_link />
-    </collision>
+    </collision> -->
     <inertial>
       <xacro:insert_inertia_r_sho_pitch_link />
@@ -43,7 +40,7 @@
       <xacro:insert_mesh_r_sho_roll_link />
     </visual>
-    <collision>
+    <!-- <collision>
       <xacro:insert_mesh_r_sho_roll_link />
-    </collision>
+    </collision> -->
     <inertial>
       <xacro:insert_inertia_r_sho_roll_link />
@@ -65,7 +62,7 @@
       <xacro:insert_mesh_r_el_link />
     </visual>
-    <collision>
+    <!-- <collision>
       <xacro:insert_mesh_r_el_link />
-    </collision>
+    </collision> -->
     <inertial>
       <xacro:insert_inertia_r_el_link />

File: op3_description/urdf/robotis_op3.structure.rleg.xacro (robot description, xacro)
@@ -1,7 +1,4 @@
 <?xml version="1.0" ?>
 <robot xmlns:xacro="http://ros.org/wiki/xacro">
-  <!--
-  <xacro:property name="pi" value="3.141592654" />
-  -->
   <!-- right leg -->
   <xacro:macro name="robotis_op3_r_leg" params="parent">
@@ -21,7 +18,7 @@
       <xacro:insert_mesh_r_hip_yaw_link />
     </visual>
-    <collision>
+    <!-- <collision>
       <xacro:insert_mesh_r_hip_yaw_link />
-    </collision>
+    </collision> -->
     <inertial>
       <xacro:insert_inertia_r_hip_yaw_link />
@@ -43,7 +40,7 @@
       <xacro:insert_mesh_r_hip_roll_link />
     </visual>
-    <collision>
+    <!-- <collision>
       <xacro:insert_mesh_r_hip_roll_link />
-    </collision>
+    </collision> -->
     <inertial>
       <xacro:insert_inertia_r_hip_roll_link />
@@ -65,7 +62,7 @@
       <xacro:insert_mesh_r_hip_pitch_link />
     </visual>
-    <collision>
+    <!-- <collision>
       <xacro:insert_mesh_r_hip_pitch_link />
-    </collision>
+    </collision> -->
     <inertial>
       <xacro:insert_inertia_r_hip_pitch_link />
@@ -87,7 +84,7 @@
       <xacro:insert_mesh_r_knee_link />
     </visual>
-    <collision>
+    <!-- <collision>
       <xacro:insert_mesh_r_knee_link />
-    </collision>
+    </collision> -->
     <inertial>
       <xacro:insert_inertia_r_knee_link />
@@ -109,7 +106,7 @@
       <xacro:insert_mesh_r_ank_pitch_link />
     </visual>
-    <collision>
+    <!-- <collision>
       <xacro:insert_mesh_r_ank_pitch_link />
-    </collision>
+    </collision> -->
     <inertial>
       <xacro:insert_inertia_r_ank_pitch_link />
@@ -131,7 +128,7 @@
       <xacro:insert_mesh_r_ank_roll_link />
     </visual>
-    <collision>
+    <!-- <collision>
       <xacro:insert_mesh_r_ank_roll_link />
-    </collision>
+    </collision> -->
     <inertial>
       <xacro:insert_inertia_r_ank_roll_link />

File: op3_description/urdf/robotis_op3.urdf.xacro (robot description, xacro)
@@ -3,28 +3,11 @@
   <xacro:include filename="$(find op3_description)/urdf/robotis_op3.visuals.xacro" />
   <xacro:include filename="$(find op3_description)/urdf/robotis_op3.inertia.xacro" />
+  <xacro:include filename="$(find op3_description)/urdf/robotis_op3.structure.rarm.xacro" />
+  <xacro:include filename="$(find op3_description)/urdf/robotis_op3.structure.larm.xacro" />
   <xacro:include filename="$(find op3_description)/urdf/robotis_op3.structure.rleg.xacro" />
   <xacro:include filename="$(find op3_description)/urdf/robotis_op3.structure.lleg.xacro" />
-  <xacro:include filename="$(find op3_description)/urdf/robotis_op3.structure.rarm.xacro" />
-  <xacro:include filename="$(find op3_description)/urdf/robotis_op3.structure.larm.xacro" />
   <xacro:include filename="$(find op3_description)/urdf/robotis_op3.structure.head.xacro" />
-  <xacro:include filename="$(find op3_description)/urdf/robotis_op3.gazebo.xacro" />
   <xacro:include filename="$(find op3_description)/urdf/robotis_op3.transmissions.xacro" />
-  <!--
-  <xacro:include filename="$(find op3_description)/urdf/gazebo_harness.xacro" />
-  -->
-  <!-- harness link -->
-  <!--
-  <xacro:add_sim_harness harnessed_link="body_link"/>
-  -->
-<!--
-  <link name="world">
-  </link>
-  <joint name="world_fixed" type="fixed">
-    <origin xyz="0 0 0" rpy="0 0 0"/>
-    <parent link="world"/>
-    <child link="base"/>
-  </joint>
-  <link name="base">
-  </link>
+  <link name="base"/>
   <joint name="base_fixed" type="fixed">
     <origin xyz="0 0 0" rpy="0 0 0"/>
@@ -32,5 +15,4 @@
     <child link="body_link"/>
   </joint>
--->
   <!-- body link -->
   <link name="body_link">
@@ -38,17 +20,17 @@
       <xacro:insert_mesh_body_link />
     </visual>
-    <collision>
-      <xacro:insert_mesh_body_link />
-    </collision>
+  <!--    <collision> -->
+  <!--      <xacro:insert_mesh_body_link /> -->
+  <!--    </collision> -->
     <inertial>
       <xacro:insert_inertia_body_link />
     </inertial>
   </link>
+  <!-- arm link -->
+  <xacro:robotis_op3_r_arm parent="body_link" />
+  <xacro:robotis_op3_l_arm parent="body_link" />
   <!-- leg link -->
+  <xacro:robotis_op3_r_leg parent="body_link" />
   <xacro:robotis_op3_l_leg parent="body_link" />
-  <xacro:robotis_op3_r_leg parent="body_link" />
-  <!-- arm link -->
-  <xacro:robotis_op3_l_arm parent="body_link" />
-  <xacro:robotis_op3_r_arm parent="body_link" />
   <!-- head links -->
   <xacro:robotis_op3_head parent="body_link" />

Commit message: added simplified collision bounds

File: op3_description/urdf/robotis_op3.structure.head.xacro (robot description, xacro)
@@ -21,4 +21,10 @@
       <xacro:insert_mesh_head_pan_link />
     </collision> -->
+    <collision>
+      <origin xyz="0.003750 0.000000 0.015500" rpy="0 0 0"/>
+      <geometry>
+        <box size="0.032500 0.042000 0.031000"/>
+      </geometry>
+    </collision>
     <inertial>
       <xacro:insert_inertia_head_pan_link />
@@ -43,4 +49,10 @@
       <xacro:insert_mesh_head_tilt_link />
     </collision> -->
+    <collision>
+      <origin xyz="0.006000 -0.019000 0.027750" rpy="0 0 0"/>
+      <geometry>
+        <box size="0.044500 0.094000 0.078000"/>
+      </geometry>
+    </collision>
     <inertial>
       <xacro:insert_inertia_head_tilt_link />

File: op3_description/urdf/robotis_op3.structure.larm.xacro (robot description, xacro)
@@ -21,4 +21,10 @@
       <xacro:insert_mesh_l_sho_pitch_link />
     </collision> -->
+    <collision>
+      <origin xyz="0.000000 0.015500 -0.003750" rpy="0 0 0"/>
+      <geometry>
+        <box size="0.042000 0.031000 0.032500"/>
+      </geometry>
+    </collision>
     <inertial>
       <xacro:insert_inertia_l_sho_pitch_link />
@@ -43,4 +49,10 @@
       <xacro:insert_mesh_l_sho_roll_link />
     </collision> -->
+    <collision>
+      <origin xyz="-0.016800 0.045200 0.000700" rpy="0 0 0"/>
+      <geometry>
+        <box size="0.042400 0.112900 0.030100"/>
+      </geometry>
+    </collision>
     <inertial>
       <xacro:insert_inertia_l_sho_roll_link />
@@ -65,4 +77,10 @@
       <xacro:insert_mesh_l_el_link />
     </collision> -->
+    <collision>
+      <origin xyz="-0.019000 0.072005 0.000000" rpy="0 0 0"/>
+      <geometry>
+        <box size="0.042000 0.149010 0.030000"/>
+      </geometry>
+    </collision>
     <inertial>
       <xacro:insert_inertia_l_el_link />

File: op3_description/urdf/robotis_op3.structure.lleg.xacro (robot description, xacro)
@@ -21,4 +21,10 @@
       <xacro:insert_mesh_l_hip_yaw_link />
     </collision> -->
+    <collision>
+      <origin xyz="0.001500 0.000000 -0.015500" rpy="0 0 0"/>
+      <geometry>
+        <box size="0.045000 0.025000 0.031000"/>
+      </geometry>
+    </collision>
     <inertial>
       <xacro:insert_inertia_l_hip_yaw_link />
@@ -43,4 +49,10 @@
       <xacro:insert_mesh_l_hip_roll_link />
     </collision> -->
+    <collision>
+      <origin xyz="0.003875 0.002200 -0.012000" rpy="0 0 0"/>
+      <geometry>
+        <box size="0.079750 0.042400 0.046500"/>
+      </geometry>
+    </collision>
     <inertial>
       <xacro:insert_inertia_l_hip_roll_link />
@@ -65,4 +77,10 @@
       <xacro:insert_mesh_l_hip_pitch_link />
     </collision> -->
+    <collision>
+      <origin xyz="0.000425 -0.018800 -0.059450" rpy="0 0 0"/>
+      <geometry>
+        <box size="0.030850 0.046400 0.123900"/>
+      </geometry>
+    </collision>
     <inertial>
       <xacro:insert_inertia_l_hip_pitch_link />
@@ -87,4 +105,10 @@
       <xacro:insert_mesh_l_knee_link />
     </collision> -->
+    <collision>
+      <origin xyz="0.000000 -0.020000 -0.055000" rpy="0 0 0"/>
+      <geometry>
+        <box size="0.030000 0.044000 0.115000"/>
+      </geometry>
+    </collision>
     <inertial>
       <xacro:insert_inertia_l_knee_link />
@@ -109,4 +133,10 @@
       <xacro:insert_mesh_l_ank_pitch_link />
     </collision> -->
+    <collision>
+      <origin xyz="-0.020600 -0.016800 0.012000" rpy="0 0 0"/>
+      <geometry>
+        <box size="0.079000 0.042400 0.046500"/>
+      </geometry>
+    </collision>
     <inertial>
       <xacro:insert_inertia_l_ank_pitch_link />
@@ -131,4 +161,10 @@
       <xacro:insert_mesh_l_ank_roll_link />
     </collision> -->
+    <collision>
+      <origin xyz="0.024000 0.012500 -0.0265" rpy="0 0 0"/>
+      <geometry>
+        <box size="0.127000 0.080000 0.008"/>
+      </geometry>
+    </collision>
     <inertial>
       <xacro:insert_inertia_l_ank_roll_link />

File: op3_description/urdf/robotis_op3.structure.rarm.xacro (robot description, xacro)
@@ -21,4 +21,10 @@
       <xacro:insert_mesh_r_sho_pitch_link />
     </collision> -->
+    <collision>
+      <origin xyz="0.000000 -0.015500 -0.003750" rpy="0 0 0"/>
+      <geometry>
+        <box size="0.042000 0.031000 0.032500"/>
+      </geometry>
+    </collision>
     <inertial>
       <xacro:insert_inertia_r_sho_pitch_link />
@@ -43,4 +49,10 @@
       <xacro:insert_mesh_r_sho_roll_link />
     </collision> -->
+    <collision>
+      <origin xyz="-0.016800 -0.045200 0.000700" rpy="0 0 0"/>
+      <geometry>
+        <box size="0.042400 0.112900 0.030100"/>
+      </geometry>
+    </collision>
     <inertial>
       <xacro:insert_inertia_r_sho_roll_link />
@@ -65,4 +77,10 @@
       <xacro:insert_mesh_r_el_link />
     </collision> -->
+    <collision>
+      <origin xyz="-0.019000 -0.072005 0.000000" rpy="0 0 0"/>
+      <geometry>
+        <box size="0.042000 0.149010 0.030000"/>
+      </geometry>
+    </collision>
     <inertial>
       <xacro:insert_inertia_r_el_link />

File: op3_description/urdf/robotis_op3.structure.rleg.xacro (robot description, xacro)
@@ -21,4 +21,10 @@
       <xacro:insert_mesh_r_hip_yaw_link />
     </collision> -->
+    <collision>
+      <origin xyz="-0.001500 0.000000 -0.015500" rpy="0 0 0"/>
+      <geometry>
+        <box size="0.045000 0.025000 0.031000"/>
+      </geometry>
+    </collision>
     <inertial>
       <xacro:insert_inertia_r_hip_yaw_link />
@@ -43,4 +49,10 @@
       <xacro:insert_mesh_r_hip_roll_link />
     </collision> -->
+    <collision>
+      <origin xyz="0.003875 -0.002200 -0.012000" rpy="0 0 0"/>
+      <geometry>
+        <box size="0.079750 0.042400 0.046500"/>
+      </geometry>
+    </collision>
     <inertial>
       <xacro:insert_inertia_r_hip_roll_link />
@@ -65,4 +77,10 @@
       <xacro:insert_mesh_r_hip_pitch_link />
     </collision> -->
+    <collision>
+      <origin xyz="0.000425 0.018800 -0.059450" rpy="0 0 0"/>
+      <geometry>
+        <box size="0.030850 0.046400 0.123900"/>
+      </geometry>
+    </collision>
     <inertial>
       <xacro:insert_inertia_r_hip_pitch_link />
@@ -87,4 +105,10 @@
       <xacro:insert_mesh_r_knee_link />
     </collision> -->
+    <collision>
+      <origin xyz="0.000000 0.020000 -0.055000" rpy="0 0 0"/>
+      <geometry>
+        <box size="0.030000 0.044000 0.115000"/>
+      </geometry>
+    </collision>
     <inertial>
       <xacro:insert_inertia_r_knee_link />
@@ -109,4 +133,10 @@
       <xacro:insert_mesh_r_ank_pitch_link />
     </collision> -->
+    <collision>
+      <origin xyz="-0.020225 0.016800 0.012000" rpy="0 0 0"/>
+      <geometry>
+        <box size="0.079750 0.042400 0.046500"/>
+      </geometry>
+    </collision>
     <inertial>
       <xacro:insert_inertia_r_ank_pitch_link />
@@ -131,4 +161,10 @@
       <xacro:insert_mesh_r_ank_roll_link />
     </collision> -->
+    <collision>
+      <origin xyz="0.024000 -0.012500 -0.0265" rpy="0 0 0"/>
+      <geometry>
+        <box size="0.127000 0.080000 0.008"/>
+      </geometry>
+    </collision>
     <inertial>
       <xacro:insert_inertia_r_ank_roll_link />

File: op3_description/urdf/robotis_op3.urdf.xacro (robot description, xacro)
@@ -8,5 +8,5 @@
   <xacro:include filename="$(find op3_description)/urdf/robotis_op3.structure.lleg.xacro" />
   <xacro:include filename="$(find op3_description)/urdf/robotis_op3.structure.head.xacro" />
-  <xacro:include filename="$(find op3_description)/urdf/robotis_op3.transmissions.xacro" />
+  <xacro:include filename="$(find op3_description)/urdf/robotis_op3.gazebo.xacro" />
   <link name="base"/>
   <joint name="base_fixed" type="fixed">
@@ -23,4 +23,10 @@
   <!--      <xacro:insert_mesh_body_link /> -->
   <!--    </collision> -->
+    <collision>
+      <origin xyz="-0.016750 0 0.068250" rpy="0 0 0"/>
+      <geometry>
+        <box size="0.11 0.12 0.135"/>
+      </geometry>
+    </collision>
     <inertial>
       <xacro:insert_inertia_body_link />
