Commit message: robotis_op3.urdf.xacro, robotis_op3.gazebo.xacro 파일 수정

File: op3_description/urdf/robotis_op3.gazebo.xacro (robot description, xacro)
@@ -1,225 +1,202 @@
 <?xml version="1.0"?>
 <robot xmlns:xacro="http://ros.org/wiki/xacro">
-  <gazebo>
-    <plugin name="gazebo_ros_control" filename="libgazebo_ros_control.so">
-      <robotNamespace>/robotis_op3</robotNamespace>
-    </plugin>
-  </gazebo>
-  <!-- body link -->
-  <gazebo reference="body_link">
-    <mu1>0.2</mu1>
-    <mu2>0.2</mu2>
-    <material>Gazebo/White</material>
-    <selfCollide>false</selfCollide>
-  </gazebo>
-  <!-- left leg links -->
-  <gazebo reference="l_hip_yaw_link">
-    <mu1>0.2</mu1>
-    <mu2>0.2</mu2>
-    <material>Gazebo/White</material>
-    <selfCollide>false</selfCollide>
-  </gazebo>
-  <gazebo reference="l_hip_roll_link">
-    <mu1>0.2</mu1>
-    <mu2>0.2</mu2>
-    <material>Gazebo/White</material>
-    <selfCollide>false</selfCollide>
-  </gazebo>
-  <gazebo reference="l_hip_pitch_link">
-    <mu1>0.2</mu1>
-    <mu2>0.2</mu2>
-    <material>Gazebo/White</material>
-    <selfCollide>false</selfCollide>
-  </gazebo>
-  <gazebo reference="l_knee_link">
-    <mu1>0.2</mu1>
-    <mu2>0.2</mu2>
-    <material>Gazebo/White</material>
-    <selfCollide>false</selfCollide>
-  </gazebo>
-  <gazebo reference="l_ank_pitch_link">
-    <mu1>0.2</mu1>
-    <mu2>0.2</mu2>
-    <material>Gazebo/White</material>
-    <selfCollide>false</selfCollide>
-  </gazebo>
-  <gazebo reference="l_ank_roll_link">
-    <kp>100000.0</kp>
-    <kd>100.0</kd>
-    <mu1>1.5</mu1>
-    <mu2>1.5</mu2>
-    <fdir1>1 0 0</fdir1>
-    <maxVel>1.0</maxVel>
-    <minDepth>0.001</minDepth>
-    <material>Gazebo/White</material>
-  </gazebo>
-  <!-- right leg links -->
-  <gazebo reference="r_hip_yaw_link">
-    <mu1>0.2</mu1>
-    <mu2>0.2</mu2>
-    <material>Gazebo/White</material>
-    <selfCollide>false</selfCollide>
-  </gazebo>
-  <gazebo reference="r_hip_roll_link">
-    <mu1>0.2</mu1>
-    <mu2>0.2</mu2>
-    <material>Gazebo/White</material>
-    <selfCollide>false</selfCollide>
-  </gazebo>
-  <gazebo reference="r_hip_pitch_link">
-    <mu1>0.2</mu1>
-    <mu2>0.2</mu2>
-    <material>Gazebo/White</material>
-    <selfCollide>false</selfCollide>
-  </gazebo>
-  <gazebo reference="r_knee_link">
-    <mu1>0.2</mu1>
-    <mu2>0.2</mu2>
-    <material>Gazebo/White</material>
-    <selfCollide>false</selfCollide>
-  </gazebo>
-  <gazebo reference="r_ank_pitch_link">
-    <mu1>0.2</mu1>
-    <mu2>0.2</mu2>
-    <material>Gazebo/White</material>
-    <selfCollide>false</selfCollide>
-  </gazebo>
-  <gazebo reference="r_ank_roll_link">
-    <mu1>9000</mu1>
-    <kp>100000.0</kp>
-    <kd>100.0</kd>
-    <mu1>1.5</mu1>
-    <mu2>1.5</mu2>
-    <fdir1>1 0 0</fdir1>
-    <maxVel>1.0</maxVel>
-    <minDepth>0.001</minDepth>
-    <material>Gazebo/White</material>
-  </gazebo>
-  <gazebo reference="r_sho_pitch_link">
-    <mu1>0.2</mu1>
-    <mu2>0.2</mu2>
-    <material>Gazebo/White</material>
-    <selfCollide>false</selfCollide>
-  </gazebo>
-  <gazebo reference="r_sho_roll_link">
-    <mu1>0.2</mu1>
-    <mu2>0.2</mu2>
-    <material>Gazebo/White</material>
-    <selfCollide>false</selfCollide>
-  </gazebo>
-  <gazebo reference="r_el_link">
-    <mu1>0.2</mu1>
-    <mu2>0.2</mu2>
-    <material>Gazebo/White</material>
-    <selfCollide>false</selfCollide>
-  </gazebo>
-  <gazebo reference="l_sho_pitch_link">
-    <mu1>0.2</mu1>
-    <mu2>0.2</mu2>
-    <material>Gazebo/White</material>
-    <selfCollide>false</selfCollide>
-  </gazebo>
-  <gazebo reference="l_sho_roll_link">
-    <mu1>0.2</mu1>
-    <mu2>0.2</mu2>
-    <material>Gazebo/White</material>
-    <selfCollide>false</selfCollide>
-  </gazebo>
-  <gazebo reference="l_el_link">
-    <mu1>0.2</mu1>
-    <mu2>0.2</mu2>
-    <material>Gazebo/White</material>
-    <selfCollide>false</selfCollide>
-  </gazebo>
-  <gazebo reference="head_pan_link">
-    <mu1>0.2</mu1>
-    <mu2>0.2</mu2>
-    <material>Gazebo/White</material>
-    <selfCollide>false</selfCollide>
-  </gazebo>
-  <gazebo reference="head_tilt_link">
-    <mu1>0.2</mu1>
-    <mu2>0.2</mu2>
-    <material>Gazebo/White</material>
-    <selfCollide>false</selfCollide>
-  </gazebo>
-  <gazebo>
-  <plugin filename="gz-sim-joint-state-publisher-system" name = "gz::sim::systems::JointStatePublisher">
-    <topic>op3_gz_joint_states</topic>
-    <joint_name>r_sho_pitch</joint_name>
-    <joint_name>l_sho_pitch</joint_name>
-    <joint_name>r_sho_roll</joint_name>
-    <joint_name>l_sho_roll</joint_name>
-    <joint_name>r_el</joint_name>
-    <joint_name>l_el</joint_name>
-    <joint_name>r_hip_yaw</joint_name>
-    <joint_name>l_hip_yaw</joint_name>
-    <joint_name>r_hip_roll</joint_name>
-    <joint_name>l_hip_roll</joint_name>
-    <joint_name>r_hip_pitch</joint_name>
-    <joint_name>l_hip_pitch</joint_name>
-    <joint_name>r_knee</joint_name>
-    <joint_name>l_knee</joint_name>
-    <joint_name>r_ank_pitch</joint_name>
-    <joint_name>l_ank_pitch</joint_name>
-    <joint_name>r_ank_roll</joint_name>
-    <joint_name>l_ank_roll</joint_name>
-    <joint_name>head_pan</joint_name>
-    <joint_name>head_tilt</joint_name>
-  </plugin>
-  </gazebo>
-  <!-- head camera -->
-  <!-- <gazebo reference="cam_gazebo_link">
-    <sensor name='camera' type='camera'>
-      <pose>-0.050000 -0.010000 0.000000 -1.5708 0.000000 -3.141592</pose>
-      <camera name='__default__'>
-        <horizontal_fov>1.012300</horizontal_fov>
-        <image>
-          <width>320</width>
-          <height>200</height>
-        </image>
-        <clip>
-          <near>0.001000</near>
-          <far>100.000000</far>
-        </clip>
-      </camera>
-      <always_on>1</always_on>
-      <update_rate>30.000000</update_rate>
-      <visualize>1</visualize>
-      <plugin name="camera_controller" filename="libgazebo_ros_camera.so">
-        <alwaysOn>true</alwaysOn>
-        <updateRate>30</updateRate>
-        <cameraName>robotis_op3/camera</cameraName>
-        <imageTopicName>image_raw</imageTopicName>
-        <cameraInfoTopicName>camera_info</cameraInfoTopicName>
-        <frameName>cam_link</frameName>
-        <hackBaseline>0.07</hackBaseline>
-        <distortionK1>0.0</distortionK1>
-        <distortionK2>0.0</distortionK2>
-        <distortionK3>0.0</distortionK3>
-        <distortionT1>0.0</distortionT1>
-        <distortionT2>0.0</distortionT2>
+  <xacro:macro name="robotis_op3_gazebo">
+    <gazebo reference="body_link">
+      <mu1>0.2</mu1>
+      <mu2>0.2</mu2>
+      <material>Gazebo/White</material>
+      <selfCollide>false</selfCollide>
+    </gazebo>
+    <!-- left leg links -->
+    <gazebo reference="l_hip_yaw_link">
+      <mu1>0.2</mu1>
+      <mu2>0.2</mu2>
+      <material>Gazebo/White</material>
+      <selfCollide>false</selfCollide>
+    </gazebo>
+    <gazebo reference="l_hip_roll_link">
+      <mu1>0.2</mu1>
+      <mu2>0.2</mu2>
+      <material>Gazebo/White</material>
+      <selfCollide>false</selfCollide>
+    </gazebo>
+    <gazebo reference="l_hip_pitch_link">
+      <mu1>0.2</mu1>
+      <mu2>0.2</mu2>
+      <material>Gazebo/White</material>
+      <selfCollide>false</selfCollide>
+    </gazebo>
+    <gazebo reference="l_knee_link">
+      <mu1>0.2</mu1>
+      <mu2>0.2</mu2>
+      <material>Gazebo/White</material>
+      <selfCollide>false</selfCollide>
+    </gazebo>
+    <gazebo reference="l_ank_pitch_link">
+      <mu1>0.2</mu1>
+      <mu2>0.2</mu2>
+      <material>Gazebo/White</material>
+      <selfCollide>false</selfCollide>
+    </gazebo>
+    <gazebo reference="l_ank_roll_link">
+      <kp>100000.0</kp>
+      <kd>100.0</kd>
+      <mu1>1.5</mu1>
+      <mu2>1.5</mu2>
+      <fdir1>1 0 0</fdir1>
+      <maxVel>1.0</maxVel>
+      <minDepth>0.001</minDepth>
+      <material>Gazebo/White</material>
+    </gazebo>
+    <!-- right leg links -->
+    <gazebo reference="r_hip_yaw_link">
+      <mu1>0.2</mu1>
+      <mu2>0.2</mu2>
+      <material>Gazebo/White</material>
+      <selfCollide>false</selfCollide>
+    </gazebo>
+    <gazebo reference="r_hip_roll_link">
+      <mu1>0.2</mu1>
+      <mu2>0.2</mu2>
+      <material>Gazebo/White</material>
+      <selfCollide>false</selfCollide>
+    </gazebo>
+    <gazebo reference="r_hip_pitch_link">
+      <mu1>0.2</mu1>
+      <mu2>0.2</mu2>
+      <material>Gazebo/White</material>
+      <selfCollide>false</selfCollide>
+    </gazebo>
+    <gazebo reference="r_knee_link">
+      <mu1>0.2</mu1>
+      <mu2>0.2</mu2>
+      <material>Gazebo/White</material>
+      <selfCollide>false</selfCollide>
+    </gazebo>
+    <gazebo reference="r_ank_pitch_link">
+      <mu1>0.2</mu1>
+      <mu2>0.2</mu2>
+      <material>Gazebo/White</material>
+      <selfCollide>false</selfCollide>
+    </gazebo>
+    <gazebo reference="r_ank_roll_link">
+      <mu1>9000</mu1>
+      <kp>100000.0</kp>
+      <kd>100.0</kd>
+      <mu1>1.5</mu1>
+      <mu2>1.5</mu2>
+      <fdir1>1 0 0</fdir1>
+      <maxVel>1.0</maxVel>
+      <minDepth>0.001</minDepth>
+      <material>Gazebo/White</material>
+    </gazebo>
+    <gazebo reference="r_sho_pitch_link">
+      <mu1>0.2</mu1>
+      <mu2>0.2</mu2>
+      <material>Gazebo/White</material>
+      <selfCollide>false</selfCollide>
+    </gazebo>
+    <gazebo reference="r_sho_roll_link">
+      <mu1>0.2</mu1>
+      <mu2>0.2</mu2>
+      <material>Gazebo/White</material>
+      <selfCollide>false</selfCollide>
+    </gazebo>
+    <gazebo reference="r_el_link">
+      <mu1>0.2</mu1>
+      <mu2>0.2</mu2>
+      <material>Gazebo/White</material>
+      <selfCollide>false</selfCollide>
+    </gazebo>
+    <gazebo reference="l_sho_pitch_link">
+      <mu1>0.2</mu1>
+      <mu2>0.2</mu2>
+      <material>Gazebo/White</material>
+      <selfCollide>false</selfCollide>
+    </gazebo>
+    <gazebo reference="l_sho_roll_link">
+      <mu1>0.2</mu1>
+      <mu2>0.2</mu2>
+      <material>Gazebo/White</material>
+      <selfCollide>false</selfCollide>
+    </gazebo>
+    <gazebo reference="l_el_link">
+      <mu1>0.2</mu1>
+      <mu2>0.2</mu2>
+      <material>Gazebo/White</material>
+      <selfCollide>false</selfCollide>
+    </gazebo>
+    <gazebo reference="head_pan_link">
+      <mu1>0.2</mu1>
+      <mu2>0.2</mu2>
+      <material>Gazebo/White</material>
+      <selfCollide>false</selfCollide>
+    </gazebo>
+    <gazebo reference="head_tilt_link">
+      <mu1>0.2</mu1>
+      <mu2>0.2</mu2>
+      <material>Gazebo/White</material>
+      <selfCollide>false</selfCollide>
+    </gazebo>
+    <gazebo>
+      <plugin filename="gz-sim-joint-state-publisher-system" name = "gz::sim::systems::JointStatePublisher">
+        <topic>op3_gz_joint_states</topic>
+        <joint_name>r_sho_pitch</joint_name>
+        <joint_name>l_sho_pitch</joint_name>
+        <joint_name>r_sho_roll</joint_name>
+        <joint_name>l_sho_roll</joint_name>
+        <joint_name>r_el</joint_name>
+        <joint_name>l_el</joint_name>
+        <joint_name>r_hip_yaw</joint_name>
+        <joint_name>l_hip_yaw</joint_name>
+        <joint_name>r_hip_roll</joint_name>
+        <joint_name>l_hip_roll</joint_name>
+        <joint_name>r_hip_pitch</joint_name>
+        <joint_name>l_hip_pitch</joint_name>
+        <joint_name>r_knee</joint_name>
+        <joint_name>l_knee</joint_name>
+        <joint_name>r_ank_pitch</joint_name>
+        <joint_name>l_ank_pitch</joint_name>
+        <joint_name>r_ank_roll</joint_name>
+        <joint_name>l_ank_roll</joint_name>
+        <joint_name>head_pan</joint_name>
+        <joint_name>head_tilt</joint_name>
       </plugin>
-    </sensor>
-  </gazebo> -->
-  <!-- imu sensor -->
-  <!-- <gazebo reference="body_link">
-    <gravity>true</gravity>
-    <sensor name="imu_sensor" type="imu">
-      <always_on>true</always_on>
-      <update_rate>100</update_rate>
-      <visualize>true</visualize>
-      <topic>__default_topic__</topic>
-      <plugin filename="libgazebo_ros_imu_sensor.so" name="imu_plugin">
-        <topicName>robotis_op3/imu</topicName>
-        <bodyName>body_link</bodyName>
-        <updateRateHZ>10.0</updateRateHZ>
-        <gaussianNoise>0.0</gaussianNoise>
-        <xyzOffset>0 0 0</xyzOffset>
-        <rpyOffset>0 0 0</rpyOffset>
-        <frameName>body_link</frameName>
-      </plugin>
-      <pose>0 0 0 0 0 0</pose>
-    </sensor>
-  </gazebo> -->
+    </gazebo>
+    <gazebo reference="cam_gazebo_link">
+      <sensor name='camera' type='camera'>
+        <gz_frame_id>cam_gazebo_link</gz_frame_id>
+        <camera name='__default__'>
+          <horizontal_fov>1.012300</horizontal_fov>
+          <image>
+            <width>320</width>
+            <height>200</height>
+          </image>
+          <clip>
+            <near>0.001000</near>
+            <far>100.000000</far>
+          </clip>
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
File: op3_description/urdf/robotis_op3.urdf.xacro (robot description, xacro)
@@ -8,6 +8,6 @@
   <xacro:include filename="$(find op3_description)/urdf/robotis_op3.structure.lleg.xacro" />
   <xacro:include filename="$(find op3_description)/urdf/robotis_op3.structure.head.xacro" />
-  <!-- <xacro:include filename="$(find op3_description)/urdf/robotis_op3.gazebo.xacro" />  -->
-  <xacro:include filename="$(find op3_gazebo_ros2)/gazebo/robotis_op3.gazebo.xacro" />
+  <xacro:include filename="$(find op3_description)/urdf/robotis_op3.gazebo.xacro" />
+  <!-- <xacro:include filename="$(find op3_gazebo_ros2)/gazebo/robotis_op3.gazebo.xacro" />  -->
   <link name="base"/>
   <joint name="base_fixed" type="fixed">
